File: pcb/power_switch_controller.sch (KiCad schematic (older format))
At the start: 1 part

Commit message: Initial design setup.
Parts:
- removed SHIELD?: ARDUINO_MEGA_SHIELD_FULL, symbol ARDUINO_MEGA_SHIELD_FULL
- added ARDUINO1: ARDUINO_MEGA, aalborg_mfc_interface:ARDUINO_MEGA_SHIELD, symbol ARDUINO_MEGA
- added C1, C2, C3: 10uF, aalborg_mfc_interface:SM1210, symbol 10uF
- added C4, C5: 0.1uF, aalborg_mfc_interface:SM1210, symbol 0.1uF
- added D1: LED_24V, aalborg_mfc_interface:LED_555-3XXX, symbol LED_24V
- added E?: ENCODER_C14, power_switch_controller:Micro-MaTch_6_SMD, symbol ENCODER_C14
- added P1: PWR_JACK_2.5x5.5, aalborg_mfc_interface:DCJACK_2PIN_HIGHCURRENT, symbol PWR_JACK_2.5x5.5
- added P2: HEADER_01X03, aalborg_mfc_interface:Header_Shrouded_3_Pin, symbol HEADER_01X03
- added R1, R2: 5.11k, aalborg_mfc_interface:SM1210, symbol 5.11k
- added REG1: CONV_DC_DC_12V_1A, aalborg_mfc_interface:DC_DC_CONV_R78C, symbol CONV_DC_DC_12V_1A
- added U1: MAX6817, aalborg_mfc_interface:MAX6817, symbol MAX6817
- added U2: TLE723X, power_switch_controller:TLE723X, symbol TLE723X
Connections:
- net labels added: D_ENC_BTN, ENC_A, ENC_B, ENC_BTN, OUT0, OUT1, OUT2, OUT3, OUT4, OUT5, OUT6, OUT7, SO1, TX3, VAA, V_IN
- wire segments 12 -> 89

Commit message: Made design changes preparing for version 1.0.
Parts:
- added C6: 0.1uF, power_switch_controller:SM1210, symbol 0.1uF
- added D10, D11, D12, D13, D14, D15, D16, D17, D2, D3, D4, D5, D6, D7, D8, D9: LED_24V, power_switch_controller:LED_555-3XXX, symbol LED_24V
- added RJ1, RJ2: RJ45_DOUBLE, power_switch_controller:RJ45_2PORT_2ROW, symbol RJ45_DOUBLE
- added S1, S10, S11, S12, S13, S14, S15, S16, S2, S3, S4, S5, S6, S7, S8, S9: HEADER_01X02_POL, power_switch_controller:Header_Shrouded_2_Pin, symbol HEADER_01X02_POL
- added SW1: SPST_SERIES_M, power_switch_controller:SPST_SERIES_M, symbol SPST_SERIES_M
- added U3: TLE723X, power_switch_controller:TLE723X, symbol TLE723X
- ARDUINO1: footprint aalborg_mfc_interface:ARDUINO_MEGA_SHIELD -> power_switch_controller:ARDUINO_MEGA_SHIELD
- C1, C2, C3, C4, C5, R1, R2: footprint aalborg_mfc_interface:SM1210 -> power_switch_controller:SM1210
- D1: footprint aalborg_mfc_interface:LED_555-3XXX -> power_switch_controller:LED_555-3XXX
- P1: footprint aalborg_mfc_interface:DCJACK_2PIN_HIGHCURRENT -> power_switch_controller:DCJACK_2PIN_HIGHCURRENT
- P2: footprint aalborg_mfc_interface:Header_Shrouded_3_Pin -> power_switch_controller:Header_Shrouded_3_Pin
- REG1: footprint aalborg_mfc_interface:DC_DC_CONV_R78C -> power_switch_controller:DC_DC_CONV_R78C
- U1: footprint aalborg_mfc_interface:MAX6817 -> power_switch_controller:MAX6817
- gave numbers to parts that had none: 1
Connections:
- net labels added: LED_PWR, OUT10, OUT11, OUT12, OUT13, OUT14, OUT15, OUT8, OUT9
- wire segments 89 -> 228
- no-connect marks 76 -> 73
Other:
- moved on the sheet: C1, C2, C3, C4, D1, P1, P2, REG1, U1

Commit message: Changed connectors to 2x16 header.
Parts:
- removed RJ1, RJ2: RJ45_DOUBLE, power_switch_controller:RJ45_2PORT_2ROW, symbol RJ45_DOUBLE
- removed S1, S10, S11, S12, S13, S14, S15, S16, S2, S3, S4, S5, S6, S7, S8, S9: HEADER_01X02_POL, power_switch_controller:Header_Shrouded_2_Pin, symbol HEADER_01X02_POL
- added P3: HEADER_02X16, power_switch_controller:HEADER_02x32, symbol HEADER_02X16
Connections:
- net labels added: SI1
- net labels removed: SO1
- wire segments 228 -> 191
Other:
- moved on the sheet: ARDUINO1, C3, C5, C6, D10, D11, D12, D13, D14, D15, D16, D17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

Commit message: Moved components on pcb.
Parts:
- added P3: BNC_DOUBLE_RA, power_switch_controller:BNC_DOUBLE, symbol BNC_DOUBLE_RA
- added R3: 5.11k, power_switch_controller:SM1210, symbol 5.11k
- renumbered P3 to P4
Connections:
- net GND: now also P3.2 (P2), P3.4 (P4), R3.1
- net LED_PWR: now also U1.3 (IN2), R3.2
- net D_LED_PWR: now reaches ARDUINO1.18 (D18/TX1/INT3/PD3)
- net D_LED_PWR: now also U1.4 (OUT2)
- net BNC_B: now reaches ARDUINO1.20B (D20/SDA/INT1/PD1)
- net BNC_B: now also P3.3 (P3)
- net BNC_A: now reaches ARDUINO1.21B (D21/SCL/INT0/PD0)
- net BNC_A: now also P3.1 (P1)
- no-connect marks 73 -> 68
Changed lines of the file:
@@
 NoConn ~ 1350 3950
 NoConn ~ 1350 4050
-NoConn ~ 1350 4200
 NoConn ~ 1350 4850
 NoConn ~ 1350 4950
@@
 NoConn ~ 1350 5500
 NoConn ~ 1350 5600
-NoConn ~ 3550 800
-NoConn ~ 3550 900
 NoConn ~ 3550 1000
 NoConn ~ 3550 1100
-NoConn ~ 3550 1200
 NoConn ~ 3550 1300
 NoConn ~ 3550 1400
@@
 NoConn ~ 3550 3000
 NoConn ~ 3550 3100
-NoConn ~ 3550 3200
-NoConn ~ 3550 3400
-NoConn ~ 3550 3500
 NoConn ~ 3550 3750
 NoConn ~ 3550 3850
@@
 Wire Wire Line
 	3850 7500 3850 7650
-NoConn ~ 3450 7200
-NoConn ~ 4250 7200
 $Comp
 L GND #PWR016
@@
 F 6 "RES SMD 5.11K OHM 1% 1/2W 1210" V 3030 7350 60  0001 C CNN "Description"
 	1    2650 7050
-	1    0    0    -1
-$EndComp
-$Comp
-L ARDUINO_MEGA ARDUINO1
-U 1 1 5489C516
-P 2500 3350
-F 0 "ARDUINO1" H 2550 6100 60  0000 C CNN
-F 1 "ARDUINO_MEGA" H 2500 650 60  0000 C CNN
-F 2 "power_switch_controller:ARDUINO_MEGA_SHIELD" H 2450 6000 60  0001 C CNN
-F 3 "" H 2550 6100 60  0000 C CNN
-F 4 "digikey" H 2650 6200 60  0001 C CNN "Vendor"
-F 5 "1050-1018-ND" H 2750 6300 60  0001 C CNN "PartNumber"
-F 6 "BOARD MCU MEGA2560" H 2850 6400 60  0001 C CNN "Description"
-	1    2500 3350
 	1    0    0    -1
 $EndComp
@@
 	5100 700  5100 800
 Wire Wire Line
-	5100 1800 5100 1900
+	5100 1800 5100 2100
 Wire Wire Line
 	5100 1900 5200 1900
@@
 NoConn ~ 1350 5800
 $Comp
-L HEADER_02X16 P3
+L HEADER_02X16 P4
 U 1 1 54ACCE04
 P 5050 3400
-F 0 "P3" H 5050 4250 50  0000 C CNN
+F 0 "P4" H 5050 4250 50  0000 C CNN
 F 1 "HEADER_02X16" V 5050 3400 50  0000 C CNN
 F 2 "power_switch_controller:HEADER_02x32" H 5050 2300 60  0001 C CNN
@@
 $EndComp
 Wire Wire Line
-	4800 4150 4700 4150
-Wire Wire Line
-	4700 4150 4700 2550
+	4700 4150 4800 4150
+Wire Wire Line
+	4700 2550 4700 4150
 Wire Wire Line
 	4800 4050 4700 4050
@@
 Text Label 5400 4150 0    60   ~ 0
 OUT15
+NoConn ~ 3550 3400
+NoConn ~ 3550 3500
+$Comp
+L ARDUINO_MEGA ARDUINO1
+U 1 1 54AD3990
+P 2500 3350
+F 0 "ARDUINO1" H 2550 6100 60  0000 C CNN
+F 1 "ARDUINO_MEGA" H 2500 650 60  0000 C CNN
+F 2 "power_switch_controller:ARDUINO_MEGA_SHIELD" H 2450 6000 60  0001 C CNN
+F 3 "" H 2550 6100 60  0000 C CNN
+F 4 "digikey" H 2650 6200 60  0001 C CNN "Vendor"
+F 5 "1050-1018-ND" H 2750 6300 60  0001 C CNN "PartNumber"
+F 6 "BOARD MCU MEGA2560" H 2850 6400 60  0001 C CNN "Description"
+	1    2500 3350
+	1    0    0    -1
+$EndComp
+$Comp
+L 5.11k R3
+U 1 1 54AD64AC
+P 5450 2100
+F 0 "R3" V 5530 2100 40  0000 C CNN
+F 1 "5.11k" V 5457 2101 40  0000 C CNN
+F 2 "power_switch_controller:SM1210" V 5380 2100 30  0001 C CNN
+F 3 "" H 5450 2100 30  0000 C CNN
+F 4 "digikey" V 5630 2200 60  0001 C CNN "Vendor"
+F 5 "P5.11KAACT-ND" V 5730 2300 60  0001 C CNN "PartNumber"
+F 6 "RES SMD 5.11K OHM 1% 1/2W 1210" V 5830 2400 60  0001 C CNN "Description"
+	1    5450 2100
+	0    1    1    0
+$EndComp
+$Comp
+L GND #PWR024
+U 1 1 54AD735F
+P 5800 2200
+F 0 "#PWR024" H 5800 1950 60  0001 C CNN
+F 1 "GND" H 5800 2050 60  0000 C CNN
+F 2 "" H 5800 2200 60  0000 C CNN
+F 3 "" H 5800 2200 60  0000 C CNN
+	1    5800 2200
+	1    0    0    -1
+$EndComp
+Wire Wire Line
+	5100 2100 5200 2100
+Connection ~ 5100 1900
+Wire Wire Line
+	5700 2100 5800 2100
+Wire Wire Line
+	5800 2100 5800 2200
+Wire Wire Line
+	3450 7200 3050 7200
+Text Label 3050 7200 0    60   ~ 0
+LED_PWR
+Wire Wire Line
+	4250 7200 4450 7200
+Text Label 4450 7200 0    60   ~ 0
+D_LED_PWR
+Wire Wire Line
+	3550 3200 3750 3200
+Text Label 3750 3200 0    60   ~ 0
+D_LED_PWR
+$Comp
+L GND #PWR025
+U 1 1 54AD9AEC
+P 8250 6350
+F 0 "#PWR025" H 8250 6100 60  0001 C CNN
+F 1 "GND" H 8250 6200 60  0000 C CNN
+F 2 "" H 8250 6350 60  0000 C CNN
+F 3 "" H 8250 6350 60  0000 C CNN
+	1    8250 6350
+	1    0    0    -1
+$EndComp
+Wire Wire Line
+	8150 6100 8250 6100
+Wire Wire Line
+	8250 6100 8250 6350
+Wire Wire Line
+	8150 6200 8250 6200
+Connection ~ 8250 6200
+Wire Wire Line
+	7650 6100 7300 6100
+Wire Wire Line
+	7650 6200 7300 6200
+Text Label 7300 6100 0    60   ~ 0
+BNC_A
+Text Label 7300 6200 0    60   ~ 0
+BNC_B
+Wire Wire Line
+	3550 800  3750 800
+Wire Wire Line
+	3550 900  3750 900
+Text Label 3750 800  0    60   ~ 0
+BNC_A
+Text Label 3750 900  0    60   ~ 0
+BNC_B
+NoConn ~ 3550 1200
+$Comp
+L BNC_DOUBLE_RA P3
+U 1 1 54ADBC63
+P 7900 6150
+F 0 "P3" H 7900 6300 50  0000 C CNN
+F 1 "BNC_DOUBLE_RA" H 7900 6000 50  0000 C CNN
+F 2 "power_switch_controller:BNC_DOUBLE" H 7900 4950 60  0001 C CNN
+F 3 "" H 7900 4950 60  0000 C CNN
+F 4 "digikey" H 8000 6400 60  0001 C CNN "Vendor"
+F 5 "ACX1655-ND" H 8100 6500 60  0001 C CNN "PartNumber"
+F 6 "CONN BNC JACK R/A 75 OHM PCB" H 8200 6600 60  0001 C CNN "Description"
+	1    7900 6150
+	1    0    0    -1
+$EndComp
+NoConn ~ 1350 4200
 $EndSCHEMATC

Commit message: Finished pcb version 1.0
Parts:
- removed P4: HEADER_02X16, power_switch_controller:HEADER_02x32, symbol HEADER_02X16
- added P4, P5: HEADER_02X08, power_switch_controller:HEADER_02x08, symbol HEADER_02X08
Connections:
- net BNC_A: now also ARDUINO1.A0 (A0/PF0); no longer ARDUINO1.21B (D21/SCL/INT0/PD0)
- net BNC_B: now also ARDUINO1.10 (D10/PWM/OC2A/PCINT4/PB4); no longer ARDUINO1.20B (D20/SDA/INT1/PD1)
- net OUT0: now also P4.2 (P2)
- net OUT1: now also P4.4 (P4)
- net OUT10: now also P5.6 (P6)
- net OUT11: now also P5.8 (P8)
- net OUT12: now also P5.10 (P10)
- net OUT13: now also P5.12 (P12)
- net OUT14: now also P5.14 (P14)
- net OUT15: now also P5.16 (P16)
- net OUT2: now also P4.6 (P6)
- net OUT3: now also P4.8 (P8)
- net OUT4: now also P4.10 (P10)
- net OUT5: now also P4.12 (P12)
- net OUT6: now also P4.14 (P14)
- net OUT7: now also P4.16 (P16)
- net OUT8: now also P5.2 (P2)
- net OUT9: now also P5.4 (P4)
- net VAA: now also P4.1 (P1), P4.11 (P11), P4.13 (P13), P4.15 (P15), P4.3 (P3), P4.5 (P5), P4.7 (P7), P4.9 (P9), P5.1 (P1), P5.11 (P11), P5.13 (P13), P5.15 (P15), P5.3 (P3), P5.5 (P5), P5.7 (P7), P5.9 (P9)
Changed lines of the file:
@@
 NoConn ~ 3550 1300
 NoConn ~ 3550 1400
-NoConn ~ 3550 1500
 NoConn ~ 3550 1600
 NoConn ~ 3550 2000
@@
 Text Label 1000 1400 0    60   ~ 0
 RST
-NoConn ~ 1350 2100
 NoConn ~ 1350 2200
 NoConn ~ 3550 1700
@@
 NoConn ~ 1350 5800
 $Comp
-L HEADER_02X16 P4
-U 1 1 54ACCE04
-P 5050 3400
-F 0 "P4" H 5050 4250 50  0000 C CNN
-F 1 "HEADER_02X16" V 5050 3400 50  0000 C CNN
-F 2 "power_switch_controller:HEADER_02x32" H 5050 2300 60  0001 C CNN
-F 3 "" H 5050 2300 60  0000 C CNN
-F 4 "digikey" H 5150 4350 60  0001 C CNN "Vendor"
-F 5 "609-3368-ND" H 5250 4450 60  0001 C CNN "PartNumber"
-F 6 "CONN HEADER 32POS .100 STR 30AU" H 5350 4550 60  0001 C CNN "Description"
-	1    5050 3400
-	1    0    0    -1
-$EndComp
-$Comp
 L VAA #PWR023
 U 1 1 54ACE02B
@@
 	1    0    0    -1
 $EndComp
-Wire Wire Line
-	4700 4150 4800 4150
-Wire Wire Line
-	4700 2550 4700 4150
-Wire Wire Line
-	4800 4050 4700 4050
-Connection ~ 4700 4050
-Wire Wire Line
-	4800 3950 4700 3950
-Connection ~ 4700 3950
-Wire Wire Line
-	4800 3850 4700 3850
-Connection ~ 4700 3850
-Wire Wire Line
-	4800 3750 4700 3750
-Connection ~ 4700 3750
-Wire Wire Line
-	4800 3650 4700 3650
-Connection ~ 4700 3650
-Wire Wire Line
-	4800 3550 4700 3550
-Connection ~ 4700 3550
-Wire Wire Line
-	4800 3450 4700 3450
-Connection ~ 4700 3450
-Wire Wire Line
-	4800 3350 4700 3350
-Connection ~ 4700 3350
-Wire Wire Line
-	4800 3250 4700 3250
-Connection ~ 4700 3250
-Wire Wire Line
-	4800 3150 4700 3150
-Connection ~ 4700 3150
-Wire Wire Line
-	4800 3050 4700 3050
-Connection ~ 4700 3050
-Wire Wire Line
-	4800 2950 4700 2950
-Connection ~ 4700 2950
-Wire Wire Line
-	4800 2850 4700 2850
-Connection ~ 4700 2850
-Wire Wire Line
-	4800 2750 4700 2750
-Connection ~ 4700 2750
-Wire Wire Line
-	4800 2650 4700 2650
-Connection ~ 4700 2650
-Wire Wire Line
-	5300 2650 5400 2650
-Wire Wire Line
-	5300 2750 5400 2750
-Wire Wire Line
-	5300 2850 5400 2850
-Wire Wire Line
-	5300 2950 5400 2950
-Wire Wire Line
-	5300 3050 5400 3050
-Wire Wire Line
-	5300 3150 5400 3150
-Wire Wire Line
-	5300 3250 5400 3250
-Wire Wire Line
-	5300 3350 5400 3350
-Wire Wire Line
-	5300 3450 5400 3450
-Wire Wire Line
-	5300 3550 5400 3550
-Wire Wire Line
-	5300 3650 5400 3650
-Wire Wire Line
-	5300 3750 5400 3750
-Wire Wire Line
-	5300 3850 5400 3850
-Wire Wire Line
-	5300 3950 5400 3950
-Wire Wire Line
-	5300 4050 5400 4050
-Wire Wire Line
-	5300 4150 5400 4150
 Text Label 5400 2650 0    60   ~ 0
 OUT0
@@
 Text Label 5400 3350 0    60   ~ 0
 OUT7
-Text Label 5400 3450 0    60   ~ 0
+Text Label 5400 3850 0    60   ~ 0
 OUT8
-Text Label 5400 3550 0    60   ~ 0
+Text Label 5400 3950 0    60   ~ 0
 OUT9
-Text Label 5400 3650 0    60   ~ 0
+Text Label 5400 4050 0    60   ~ 0
 OUT10
-Text Label 5400 3750 0    60   ~ 0
+Text Label 5400 4150 0    60   ~ 0
 OUT11
-Text Label 5400 3850 0    60   ~ 0
+Text Label 5400 4250 0    60   ~ 0
 OUT12
-Text Label 5400 3950 0    60   ~ 0
+Text Label 5400 4350 0    60   ~ 0
 OUT13
-Text Label 5400 4050 0    60   ~ 0
+Text Label 5400 4450 0    60   ~ 0
 OUT14
-Text Label 5400 4150 0    60   ~ 0
+Text Label 5400 4550 0    60   ~ 0
 OUT15
 NoConn ~ 3550 3400
@@
 Text Label 7300 6200 0    60   ~ 0
 BNC_B
-Wire Wire Line
-	3550 800  3750 800
-Wire Wire Line
-	3550 900  3750 900
-Text Label 3750 800  0    60   ~ 0
-BNC_A
-Text Label 3750 900  0    60   ~ 0
+Text Label 3750 1500 0    60   ~ 0
 BNC_B
 NoConn ~ 3550 1200
@@
 $EndComp
 NoConn ~ 1350 4200
+Wire Wire Line
+	1350 2100 1000 2100
+Text Label 1000 2100 0    60   ~ 0
+BNC_A
+NoConn ~ 3550 900
+NoConn ~ 3550 800
+Wire Wire Line
+	3550 1500 3750 1500
+$Comp
+L HEADER_02X08 P4
+U 1 1 54AEE5A9
+P 5050 3000
+F 0 "P4" H 5050 3450 50  0000 C CNN
+F 1 "HEADER_02X08" V 5050 3000 50  0000 C CNN
+F 2 "power_switch_controller:HEADER_02x08" H 5050 1800 60  0001 C CNN
+F 3 "" H 5050 1800 60  0000 C CNN
+F 4 "digikey" H 5150 3550 60  0001 C CNN "Vendor"
+F 5 "A33163-ND" H 5250 3650 60  0001 C CNN "PartNumber"
+F 6 "CONN HEADER LOPRO STR 16POS GOLD" H 5350 3750 60  0001 C CNN "Description"
+	1    5050 3000
+	1    0    0    -1
+$EndComp
+Wire Wire Line
+	5400 2650 5300 2650
+Wire Wire Line
+	5400 2750 5300 2750
+Wire Wire Line
+	5400 2850 5300 2850
+Wire Wire Line
+	5400 2950 5300 2950
+Wire Wire Line
+	5400 3050 5300 3050
+Wire Wire Line
+	5400 3150 5300 3150
+Wire Wire Line
+	5400 3250 5300 3250
+Wire Wire Line
+	5400 3350 5300 3350
+Wire Wire Line
+	4800 3350 4700 3350
+Wire Wire Line
+	4700 3350 4700 2550
+Wire Wire Line
+	4800 3250 4700 3250
+Connection ~ 4700 3250
+Wire Wire Line
+	4800 3150 4700 3150
+Connection ~ 4700 3150
+Wire Wire Line
+	4800 3050 4700 3050
+Connection ~ 4700 3050
+Wire Wire Line
+	4800 2950 4700 2950
+Connection ~ 4700 2950
+Wire Wire Line
+	4800 2850 4700 2850
+Connection ~ 4700 2850
+Wire Wire Line
+	4800 2750 4700 2750
+Connection ~ 4700 2750
+Wire Wire Line
+	4800 2650 4700 2650
+Connection ~ 4700 2650
+$Comp
+L VAA #PWR?
+U 1 1 54AEFA4B
+P 4700 3750
+F 0 "#PWR?" H 4700 3600 60  0001 C CNN
+F 1 "VAA" H 4700 3900 60  0000 C CNN
+F 2 "" H 4700 3750 60  0000 C CNN
+F 3 "" H 4700 3750 60  0000 C CNN
+	1    4700 3750
+	1    0    0    -1
+$EndComp
+$Comp
+L HEADER_02X08 P5
+U 1 1 54AEFAF6
+P 5050 4200
+F 0 "P5" H 5050 4650 50  0000 C CNN
+F 1 "HEADER_02X08" V 5050 4200 50  0000 C CNN
+F 2 "power_switch_controller:HEADER_02x08" H 5050 3000 60  0001 C CNN
+F 3 "" H 5050 3000 60  0000 C CNN
+F 4 "digikey" H 5150 4750 60  0001 C CNN "Vendor"
+F 5 "A33163-ND" H 5250 4850 60  0001 C CNN "PartNumber"
+F 6 "CONN HEADER LOPRO STR 16POS GOLD" H 5350 4950 60  0001 C CNN "Description"
+	1    5050 4200
+	1    0    0    -1
+$EndComp
+Wire Wire Line
+	5400 3850 5300 3850
+Wire Wire Line
+	5400 3950 5300 3950
+Wire Wire Line
+	5400 4050 5300 4050
+Wire Wire Line
+	5400 4150 5300 4150
+Wire Wire Line
+	5400 4250 5300 4250
+Wire Wire Line
+	5400 4350 5300 4350
+Wire Wire Line
+	5400 4450 5300 4450
+Wire Wire Line
+	5400 4550 5300 4550
+Wire Wire Line
+	4800 4550 4700 4550
+Wire Wire Line
+	4700 4550 4700 3750
+Wire Wire Line
+	4800 3850 4700 3850
+Connection ~ 4700 3850
+Wire Wire Line
+	4800 3950 4700 3950
+Connection ~ 4700 3950
+Wire Wire Line
+	4800 4050 4700 4050
+Connection ~ 4700 4050
+Wire Wire Line
+	4800 4150 4700 4150
+Connection ~ 4700 4150
+Wire Wire Line
+	4800 4250 4700 4250
+Connection ~ 4700 4250
+Wire Wire Line
+	4800 4350 4700 4350
+Connection ~ 4700 4350
+Wire Wire Line
+	4800 4450 4700 4450
+Connection ~ 4700 4450
 $EndSCHEMATC
