File: pcb/power_switch_controller.sch (KiCad schematic (older format))
At the start: 63 parts, among them P1 PWR_JACK_2.5x5.5, P2 HEADER_01X03, P3 BNC_DOUBLE_RA, P4 HEADER_02X08_SMD, P5 HEADER_02X08_SMD, P6 HEADER_02X08_SMD, P7 HEADER_02X08_SMD, SW1 DPST_SERIES_M, SW2 KT_SWITCH, U1 MAX6817, U2 MAX6817, U3 TLE723X, U4 TLE723X, U5 TLE723X, U6 TLE723X

Commit message: Kicad update.
Parts:
- U1, U2: symbol MAX6817 -> MAX6817-RESCUE-power_switch_controller
Changed lines of the file:
@@
 EESchema Schematic File Version 2
+LIBS:power_switch_controller-rescue
 LIBS:power
 LIBS:device
@@
 $EndComp
 $Comp
-L MAX6817 U1
+L MAX6817-RESCUE-power_switch_controller U1
 U 1 1 5489DAE1
 P 3100 7550
@@
 $EndComp
 $Comp
-L MAX6817 U2
+L MAX6817-RESCUE-power_switch_controller U2
 U 1 1 54BF019F
 P 4950 7550

Commit message: Progress towards pcb v1.4.
Parts:
- removed C3: 10uF, power_switch_controller:SM1210, symbol 10uF
- removed C4, C5: 0.1uF, power_switch_controller:SM1210, symbol 0.1uF
- removed E1: ENCODER_C14, power_switch_controller:Micro-MaTch_6_SMD, symbol ENCODER_C14
- removed P2: HEADER_01X03, footprints:Header_3_Pin, symbol HEADER_01X03
- removed R1, R2: 5.11k, power_switch_controller:SM1210, symbol 5.11k
- removed S1: HEADER_01X02_SHR, power_switch_controller:Header_Shrouded_2_Pin, symbol HEADER_01X02_SHR
- removed SW1: DPST_SERIES_M, power_switch_controller:DPST_SERIES_M, symbol DPST_SERIES_M
- removed SW2: KT_SWITCH, power_switch_controller:KT_SWITCH, symbol KT_SWITCH
- removed U1, U2: MAX6817, power_switch_controller:MAX6817, symbol MAX6817-RESCUE-power_switch_controller
- added P2, P3, P4, P5: HEADER_01X03_SMD_RA, power_switch_controller:Header_3_Pin_SMD_RA, symbol HEADER_01X03_SMD_RA
- added P6: HEADER_01X02_SMD_RA, power_switch_controller:Header_2_Pin_SMD_RA, symbol HEADER_01X02_SMD_RA
- renumbered P6 to P10, P7 to P11, P3 to P7, P4 to P8, P5 to P9
Connections:
- net labels added: RX0, RX1, RX2, RX3, TX0, TX1, TX2
- net labels removed: BTN, D_BTN, D_ENC_BTN, D_LIGHTS, D_SWITCH, ENC_A, ENC_B, ENC_BTN, LIGHTS, SWITCH
- wire segments 346 -> 310
- no-connect marks 65 -> 62
Other:
- moved on the sheet: C1, C2, D1, P1, P7, REG1

Commit message: Updated bom.
Parts:
- added C1: 10uF, power_switch_controller:SM1210, symbol 10uF
- added SW1: SPST_SLIDE_AS, power_switch_controller:SPST_SLIDE_AS, symbol SPST_SLIDE_AS
- renumbered C1 to C2, C2 to C3, C6 to C4, C7 to C5, C8 to C6, C9 to C7, U3 to U1, U4 to U2, U5 to U3, U6 to U4
Connections:
- net GND: now also C1.2
- net LED_PWR: now also SW1.3
- net VAA: now also C1.1, SW1.1
- no-connect marks 62 -> 65
Changed lines of the file:
@@
 V_IN
 $Comp
-L GND #PWR010
+L GND #PWR08
 U 1 1 547CC155
 P 2200 7875
-F 0 "#PWR010" H 2200 7875 30  0001 C CNN
+F 0 "#PWR08" H 2200 7875 30  0001 C CNN
 F 1 "GND" H 2200 7805 30  0001 C CNN
 F 2 "" H 2200 7875 60  0000 C CNN
@@
 	2200 7775 2200 7875
 $Comp
-L VAA #PWR011
+L VAA #PWR09
 U 1 1 547CC477
 P 3175 7100
-F 0 "#PWR011" H 3175 7160 30  0001 C CNN
+F 0 "#PWR09" H 3175 7160 30  0001 C CNN
 F 1 "VAA" H 3175 7210 30  0000 C CNN
 F 2 "" H 3175 7100 60  0000 C CNN
@@
 $EndComp
 $Comp
-L GND #PWR012
+L GND #PWR010
 U 1 1 547CC4E0
 P 3775 7850
-F 0 "#PWR012" H 3775 7850 30  0001 C CNN
+F 0 "#PWR010" H 3775 7850 30  0001 C CNN
 F 1 "GND" H 3775 7780 30  0001 C CNN
 F 2 "" H 3775 7850 60  0000 C CNN
@@
 	3125 7700 3125 7750
 Wire Wire Line
-	3125 7750 4425 7750
+	2850 7750 4425 7750
 Connection ~ 3775 7750
 Wire Wire Line
@@
 	3125 7300 3125 7250
 Wire Wire Line
-	3125 7250 3375 7250
+	2850 7250 3375 7250
 Wire Wire Line
 	4175 7250 4675 7250
@@
 $EndComp
 $Comp
-L 10uF C1
+L 10uF C2
 U 1 1 548925C4
 P 3125 7500
-F 0 "C1" H 3125 7600 40  0000 L CNN
+F 0 "C2" H 3125 7600 40  0000 L CNN
 F 1 "10uF" H 3131 7415 40  0000 L CNN
 F 2 "power_switch_controller:SM1210" H 3163 7350 30  0001 C CNN
@@
 $EndComp
 $Comp
-L 10uF C2
+L 10uF C3
 U 1 1 54892682
 P 4425 7500
-F 0 "C2" H 4425 7600 40  0000 L CNN
+F 0 "C3" H 4425 7600 40  0000 L CNN
 F 1 "10uF" H 4431 7415 40  0000 L CNN
 F 2 "power_switch_controller:SM1210" H 4463 7350 30  0001 C CNN
@@
 IN
 $Comp
-L TLE723X U5
+L TLE723X U3
 U 1 1 548B22AA
 P 9550 1150
-F 0 "U5" H 9950 1650 60  0000 C CNN
+F 0 "U3" H 9950 1650 60  0000 C CNN
 F 1 "TLE723X" H 9550 1650 60  0000 C CNN
 F 2 "power_switch_controller:TLE723X" H 9850 1550 60  0001 C CNN
@@
 SI3
 $Comp
-L 0.1uF C8
+L 0.1uF C6
 U 1 1 548B293B
 P 8600 1200
-F 0 "C8" H 8600 1300 40  0000 L CNN
+F 0 "C6" H 8600 1300 40  0000 L CNN
 F 1 "0.1uF" H 8606 1115 40  0000 L CNN
 F 2 "power_switch_controller:SM1210" H 8638 1050 30  0001 C CNN
@@
 $EndComp
 $Comp
-L +5V #PWR018
+L +5V #PWR011
 U 1 1 548B2978
 P 8600 750
-F 0 "#PWR018" H 8600 600 60  0001 C CNN
+F 0 "#PWR011" H 8600 600 60  0001 C CNN
 F 1 "+5V" H 8600 890 60  0000 C CNN
 F 2 "" H 8600 750 60  0000 C CNN
@@
 Connection ~ 8600 900
 $Comp
-L GND #PWR019
+L GND #PWR012
 U 1 1 548B2B28
 P 8600 1950
-F 0 "#PWR019" H 8600 1700 60  0001 C CNN
+F 0 "#PWR012" H 8600 1700 60  0001 C CNN
 F 1 "GND" H 8600 1800 60  0000 C CNN
 F 2 "" H 8600 1950 60  0000 C CNN
@@
 OUT23
 $Comp
-L TLE723X U6
+L TLE723X U4
 U 1 1 54AADA19
 P 9550 2800
-F 0 "U6" H 9950 3300 60  0000 C CNN
+F 0 "U4" H 9950 3300 60  0000 C CNN
 F 1 "TLE723X" H 9550 3300 60  0000 C CNN
 F 2 "power_switch_controller:TLE723X" H 9850 3200 60  0001 C CNN
@@
 MISO
 $Comp
-L 0.1uF C9
+L 0.1uF C7
 U 1 1 54AADA2E
 P 8600 2850
-F 0 "C9" H 8600 2950 40  0000 L CNN
+F 0 "C7" H 8600 2950 40  0000 L CNN
 F 1 "0.1uF" H 8606 2765 40  0000 L CNN
 F 2 "power_switch_controller:SM1210" H 8638 2700 30  0001 C CNN
@@
 $EndComp
 $Comp
-L +5V #PWR020
+L +5V #PWR013
 U 1 1 54AADA34
 P 8600 2400
-F 0 "#PWR020" H 8600 2250 60  0001 C CNN
+F 0 "#PWR013" H 8600 2250 60  0001 C CNN
 F 1 "+5V" H 8600 2540 60  0000 C CNN
 F 2 "" H 8600 2400 60  0000 C CNN
@@
 Connection ~ 8600 2550
 $Comp
-L GND #PWR021
+L GND #PWR014
 U 1 1 54AADA3F
 P 8600 3600
-F 0 "#PWR021" H 8600 3350 60  0001 C CNN
+F 0 "#PWR014" H 8600 3350 60  0001 C CNN
 F 1 "GND" H 8600 3450 60  0000 C CNN
 F 2 "" H 8600 3600 60  0000 C CNN
@@
 NoConn ~ 1350 5800
 $Comp
-L VAA #PWR022
+L VAA #PWR015
 U 1 1 54ACE02B
 P 4250 950
-F 0 "#PWR022" H 4250 800 60  0001 C CNN
+F 0 "#PWR015" H 4250 800 60  0001 C CNN
 F 1 "VAA" H 4250 1100 60  0000 C CNN
 F 2 "" H 4250 950 60  0000 C CNN
@@
 $EndComp
 $Comp
-L GND #PWR024
+L GND #PWR016
 U 1 1 54AD9AEC
 P 6100 7725
-F 0 "#PWR024" H 6100 7475 60  0001 C CNN
+F 0 "#PWR016" H 6100 7475 60  0001 C CNN
 F 1 "GND" H 6100 7575 60  0000 C CNN
 F 2 "" H 6100 7725 60  0000 C CNN
@@
 	4850 1700 4800 1700
 $Comp
-L VAA #PWR025
+L VAA #PWR017
 U 1 1 54AEFA4B
 P 4250 1950
-F 0 "#PWR025" H 4250 1800 60  0001 C CNN
+F 0 "#PWR017" H 4250 1800 60  0001 C CNN
 F 1 "VAA" H 4250 2100 60  0000 C CNN
 F 2 "" H 4250 1950 60  0000 C CNN
@@
 	4850 2700 4800 2700
 $Comp
-L +5VD #PWR026
+L +5VD #PWR018
 U 1 1 54BEF7A6
 P 3800 3700
-F 0 "#PWR026" H 3800 3550 60  0001 C CNN
+F 0 "#PWR018" H 3800 3550 60  0001 C CNN
 F 1 "+5VD" H 3800 3840 60  0000 C CNN
 F 2 "" H 3800 3700 60  0000 C CNN
@@
 $EndComp
 $Comp
-L PWR_FLAG #FLG027
+L PWR_FLAG #FLG019
 U 1 1 54BEF7BA
 P 4150 3700
-F 0 "#FLG027" H 4150 3795 30  0001 C CNN
+F 0 "#FLG019" H 4150 3795 30  0001 C CNN
 F 1 "PWR_FLAG" H 4150 3880 30  0000 C CNN
 F 2 "" H 4150 3700 60  0000 C CNN
@@
 LED_PWR
 $Comp
-L TLE723X U3
+L TLE723X U1
 U 1 1 54BF6DD8
 P 7550 1150
-F 0 "U3" H 7950 1650 60  0000 C CNN
+F 0 "U1" H 7950 1650 60  0000 C CNN
 F 1 "TLE723X" H 7550 1650 60  0000 C CNN
 F 2 "power_switch_controller:TLE723X" H 7850 1550 60  0001 C CNN
@@
 SI1
 $Comp
-L 0.1uF C6
+L 0.1uF C4
 U 1 1 54BF6DED
 P 6600 1200
-F 0 "C6" H 6600 1300 40  0000 L CNN
+F 0 "C4" H 6600 1300 40  0000 L CNN
 F 1 "0.1uF" H 6606 1115 40  0000 L CNN
 F 2 "power_switch_controller:SM1210" H 6638 1050 30  0001 C CNN
@@
 $EndComp
 $Comp
-L +5V #PWR034
+L +5V #PWR020
 U 1 1 54BF6DF3
 P 6600 750
-F 0 "#PWR034" H 6600 600 60  0001 C CNN
+F 0 "#PWR020" H 6600 600 60  0001 C CNN
 F 1 "+5V" H 6600 890 60  0000 C CNN
 F 2 "" H 6600 750 60  0000 C CNN
@@
 Connection ~ 6600 900
 $Comp
-L GND #PWR035
+L GND #PWR021
 U 1 1 54BF6DFE
 P 6600 1950
-F 0 "#PWR035" H 6600 1700 60  0001 C CNN
+F 0 "#PWR021" H 6600 1700 60  0001 C CNN
 F 1 "GND" H 6600 1800 60  0000 C CNN
 F 2 "" H 6600 1950 60  0000 C CNN
@@
 OUT7
 $Comp
-L TLE723X U4
+L TLE723X U2
 U 1 1 54BF6E29
 P 7550 2800
-F 0 "U4" H 7950 3300 60  0000 C CNN
+F 0 "U2" H 7950 3300 60  0000 C CNN
 F 1 "TLE723X" H 7550 3300 60  0000 C CNN
 F 2 "power_switch_controller:TLE723X" H 7850 3200 60  0001 C CNN
@@
 SI2
 $Comp
-L 0.1uF C7
+L 0.1uF C5
 U 1 1 54BF6E3E
 P 6600 2850
-F 0 "C7" H 6600 2950 40  0000 L CNN
+F 0 "C5" H 6600 2950 40  0000 L CNN
 F 1 "0.1uF" H 6606 2765 40  0000 L CNN
 F 2 "power_switch_controller:SM1210" H 6638 2700 30  0001 C CNN
@@
 $EndComp
 $Comp
-L +5V #PWR036
+L +5V #PWR022
 U 1 1 54BF6E44
 P 6600 2400
-F 0 "#PWR036" H 6600 2250 60  0001 C CNN
+F 0 "#PWR022" H 6600 2250 60  0001 C CNN
 F 1 "+5V" H 6600 2540 60  0000 C CNN
 F 2 "" H 6600 2400 60  0000 C CNN
@@
 Connection ~ 6600 2550
 $Comp
-L GND #PWR037
+L GND #PWR023
 U 1 1 54BF6E4F
 P 6600 3600
-F 0 "#PWR037" H 6600 3350 60  0001 C CNN
+F 0 "#PWR023" H 6600 3350 60  0001 C CNN
 F 1 "GND" H 6600 3450 60  0000 C CNN
 F 2 "" H 6600 3600 60  0000 C CNN
@@
 $EndComp
 $Comp
-L VAA #PWR038
+L VAA #PWR024
 U 1 1 54BFF1C6
 P 5200 950
-F 0 "#PWR038" H 5200 800 60  0001 C CNN
+F 0 "#PWR024" H 5200 800 60  0001 C CNN
 F 1 "VAA" H 5200 1100 60  0000 C CNN
 F 2 "" H 5200 950 60  0000 C CNN
@@
 	5800 1700 5750 1700
 $Comp
-L VAA #PWR039
+L VAA #PWR025
 U 1 1 54BFF1E4
 P 5200 1950
-F 0 "#PWR039" H 5200 1800 60  0001 C CNN
+F 0 "#PWR025" H 5200 1800 60  0001 C CNN
 F 1 "VAA" H 5200 2100 60  0000 C CNN
 F 2 "" H 5200 1950 60  0000 C CNN
@@
 NoConn ~ 1350 4650
 $Comp
-L GND #PWR?
+L GND #PWR026
 U 1 1 56CE6D1F
 P 5825 3175
-F 0 "#PWR?" H 5825 2925 60  0001 C CNN
+F 0 "#PWR026" H 5825 2925 60  0001 C CNN
 F 1 "GND" H 5825 3025 60  0000 C CNN
 F 2 "" H 5825 3175 60  0000 C CNN
@@
 $EndComp
 $Comp
-L +5VD #PWR?
+L +5VD #PWR027
 U 1 1 56CF0A59
 P 3200 6450
-F 0 "#PWR?" H 3200 6300 60  0001 C CNN
+F 0 "#PWR027" H 3200 6300 60  0001 C CNN
 F 1 "+5VD" H 3200 6590 60  0000 C CNN
 F 2 "" H 3200 6450 60  0000 C CNN
@@
 $EndComp
 $Comp
-L GND #PWR?
+L GND #PWR028
 U 1 1 56CF0FA4
 P 3200 6650
-F 0 "#PWR?" H 3200 6650 30  0001 C CNN
+F 0 "#PWR028" H 3200 6650 30  0001 C CNN
 F 1 "GND" H 3200 6580 30  0001 C CNN
 F 2 "" H 3200 6650 60  0000 C CNN
@@
 Wire Wire Line
 	3200 6600 3200 6650
+$Comp
+L VAA #PWR029
+U 1 1 56CF9310
+P 1575 7225
+F 0 "#PWR029" H 1575 7285 30  0001 C CNN
+F 1 "VAA" H 1575 7335 30  0000 C CNN
+F 2 "" H 1575 7225 60  0000 C CNN
+F 3 "" H 1575 7225 60  0000 C CNN
+	1    1575 7225
+	1    0    0    -1
+$EndComp
+Wire Wire Line
+	1575 7775 1575 7875
+Text Label 1575 7875 0    60   ~ 0
+LED_PWR
+NoConn ~ 3550 3400
+NoConn ~ 3550 3500
+NoConn ~ 1350 5150
+Wire Wire Line
+	1575 7225 1575 7275
+$Comp
+L SPST_SLIDE_AS SW1
+U 1 1 56CFEB9B
+P 1575 7525
+F 0 "SW1" H 1500 7450 40  0000 L CNN
+F 1 "SPST_SLIDE_AS" H 1350 7625 40  0000 L CNN
+F 2 "power_switch_controller:SPST_SLIDE_AS" H 1475 7325 60  0001 C CNN
+F 3 "" H 1575 7475 60  0000 C CNN
+F 4 "digikey" H 1675 7725 60  0001 C CNN "Vendor"
+F 5 "360-2610-ND" H 1775 7825 60  0001 C CNN "PartNumber"
+F 6 "SWITCH SLIDE SPST 0.4VA 28V" H 1875 7925 60  0001 C CNN "Description"
+	1    1575 7525
+	0    1    1    0
+$EndComp
+$Comp
+L 10uF C1
+U 1 1 56D083E8
+P 2850 7500
+F 0 "C1" H 2850 7600 40  0000 L CNN
+F 1 "10uF" H 2856 7415 40  0000 L CNN
+F 2 "power_switch_controller:SM1210" H 2888 7350 30  0001 C CNN
+F 3 "" H 2850 7500 60  0000 C CNN
+F 4 "digikey" H 2950 7700 60  0001 C CNN "Vendor"
+F 5 "445-4536-1-ND" H 3050 7800 60  0001 C CNN "PartNumber"
+F 6 "CAP CER 10UF 50V 10% X7S 1210" H 3150 7900 60  0001 C CNN "Description"
+	1    2850 7500
+	1    0    0    -1
+$EndComp
+Wire Wire Line
+	2850 7250 2850 7300
+Connection ~ 3125 7250
+Wire Wire Line
+	2850 7750 2850 7700
+Connection ~ 3125 7750
 $EndSCHEMATC

Commit message: Finished pcb v1.5.
Parts:
- removed U1, U2, U3, U4: TLE723X, power_switch_controller:TLE723X, symbol TLE723X
- added U1, U2, U3, U4: TLE7230R, power_switch_controller:PG-DSO-36, symbol TLE7230R
Connections:
- net +5V: now also U1.25 (VDO), U1.8 (VS), U2.25 (VDO), U2.8 (VS), U3.25 (VDO), U3.8 (VS), U4.25 (VDO), U4.8 (VS)
- net +5VD: no longer P6.2 (P2)
- net CS: now also U1.10 (CS), U2.10 (CS), U3.10 (CS), U4.10 (CS)
- net GND: now also U1.1 (GND), U1.12 (IN3), U1.13 (IN4), U1.18 (GND), U1.19 (GND), U1.36 (GND), U1.6 (IN1), U1.7 (IN2), U2.1 (GND), U2.12 (IN3), U2.13 (IN4), U2.18 (GND), U2.19 (GND), U2.36 (GND), U2.6 (IN1), U2.7 (IN2), U3.1 (GND), U3.12 (IN3), U3.13 (IN4), U3.18 (GND), U3.19 (GND), U3.36 (GND), U3.6 (IN1), U3.7 (IN2), U4.1 (GND), U4.12 (IN3), U4.13 (IN4), U4.18 (GND), U4.19 (GND), U4.36 (GND), U4.6 (IN1), U4.7 (IN2)
- net MISO: now also U4.27 (SO)
- net MOSI: now also U1.29 (SI)
- net OUT0: now also U1.4 (OUT1)
- net OUT1: now also U1.5 (OUT2)
- net OUT10: now also U2.14 (OUT3)
- net OUT11: now also U2.15 (OUT4)
- net OUT12: now also U2.22 (OUT5)
- net OUT13: now also U2.23 (OUT6)
- net OUT14: now also U2.32 (OUT7)
- net OUT15: now also U2.33 (OUT8)
- net OUT16: now also U3.4 (OUT1)
- net OUT17: now also U3.5 (OUT2)
- net OUT18: now also U3.14 (OUT3)
- net OUT19: now also U3.15 (OUT4)
- net OUT2: now also U1.14 (OUT3)
- net OUT20: now also U3.22 (OUT5)
- net OUT21: now also U3.23 (OUT6)
- net OUT22: now also U3.32 (OUT7)
- net OUT23: now also U3.33 (OUT8)
- net OUT24: now also U4.4 (OUT1)
- net OUT25: now also U4.5 (OUT2)
- net OUT26: now also U4.14 (OUT3)
- net OUT27: now also U4.15 (OUT4)
- net OUT28: now also U4.22 (OUT5)
- net OUT29: now also U4.23 (OUT6)
- net OUT3: now also U1.15 (OUT4)
- net OUT30: now also U4.32 (OUT7)
- net OUT31: now also U4.33 (OUT8)
- net OUT4: now also U1.22 (OUT5)
- net OUT5: now also U1.23 (OUT6)
- net OUT6: now also U1.32 (OUT7)
- net OUT7: now also U1.33 (OUT8)
- net OUT8: now also U2.4 (OUT1)
- net OUT9: now also U2.5 (OUT2)
- net SCK: now also U1.28 (SCLK), U2.28 (SCLK), U3.28 (SCLK), U4.28 (SCLK)
- net VAA: now also P6.2 (P2)
- net RESET: now reaches ARDUINO1.44 (D44/PWM/OC5C/PL5)
- net RESET: now also U1.9 (RST), U2.9 (RST), U3.9 (RST), U4.9 (RST)
- net RST: no longer names the net of ARDUINO1.RST
- new net SO1: U1.27 (SO), U2.29 (SI)
- new net SO2: U2.27 (SO), U3.29 (SI)
- new net SO3: U3.27 (SO), U4.29 (SI)
- no-connect marks 65 -> 73
Other:
- moved on the sheet: C5, C7

Commit message: Updated discontinued part.
Parts:
- P10, P11, P8, P9: Description CONN HEADER LO-PRO 16POS AU SMD -> CONN HEADR 2.54MM 16POS GOLD SMD; PartNumber HSL16H-ND -> S9187-ND
Changed lines of the file:
@@
 Connection ~ 4250 1100
-$Comp
-L HEADER_02X08_SMD P8
-U 1 1 54BFE706
-P 4550 1350
-F 0 "P8" H 4550 1800 50  0000 C CNN
-F 1 "HEADER_02X08_SMD" V 4550 1350 50  0000 C CNN
-F 2 "power_switch_controller:HEADER_02x08_SMD" H 4550 150 60  0001 C CNN
-F 3 "" H 4550 150 60  0000 C CNN
-F 4 "digikey" H 4650 1900 60  0001 C CNN "Vendor"
-F 5 "HSL16H-ND" H 4750 2000 60  0001 C CNN "PartNumber"
-F 6 "CONN HEADER LO-PRO 16POS AU SMD" H 4850 2100 60  0001 C CNN "Description"
-	1    4550 1350
-	1    0    0    -1
-$EndComp
-$Comp
-L HEADER_02X08_SMD P9
-U 1 1 54BFEC24
-P 4550 2350
-F 0 "P9" H 4550 2800 50  0000 C CNN
-F 1 "HEADER_02X08_SMD" V 4550 2350 50  0000 C CNN
-F 2 "power_switch_controller:HEADER_02x08_SMD" H 4550 1150 60  0001 C CNN
-F 3 "" H 4550 1150 60  0000 C CNN
-F 4 "digikey" H 4650 2900 60  0001 C CNN "Vendor"
-F 5 "HSL16H-ND" H 4750 3000 60  0001 C CNN "PartNumber"
-F 6 "CONN HEADER LO-PRO 16POS AU SMD" H 4850 3100 60  0001 C CNN "Description"
-	1    4550 2350
-	1    0    0    -1
-$EndComp
 $Comp
 L VAA #PWR024
@@
 	5250 1100 5200 1100
 Connection ~ 5200 1100
-$Comp
-L HEADER_02X08_SMD P10
-U 1 1 54BFF215
-P 5500 1350
-F 0 "P10" H 5500 1800 50  0000 C CNN
-F 1 "HEADER_02X08_SMD" V 5500 1350 50  0000 C CNN
-F 2 "power_switch_controller:HEADER_02x08_SMD" H 5500 150 60  0001 C CNN
-F 3 "" H 5500 150 60  0000 C CNN
-F 4 "digikey" H 5600 1900 60  0001 C CNN "Vendor"
-F 5 "HSL16H-ND" H 5700 2000 60  0001 C CNN "PartNumber"
-F 6 "CONN HEADER LO-PRO 16POS AU SMD" H 5800 2100 60  0001 C CNN "Description"
-	1    5500 1350
-	1    0    0    -1
-$EndComp
-$Comp
-L HEADER_02X08_SMD P11
-U 1 1 54BFF21E
-P 5500 2350
-F 0 "P11" H 5500 2800 50  0000 C CNN
-F 1 "HEADER_02X08_SMD" V 5500 2350 50  0000 C CNN
-F 2 "power_switch_controller:HEADER_02x08_SMD" H 5500 1150 60  0001 C CNN
-F 3 "" H 5500 1150 60  0000 C CNN
-F 4 "digikey" H 5600 2900 60  0001 C CNN "Vendor"
-F 5 "HSL16H-ND" H 5700 3000 60  0001 C CNN "PartNumber"
-F 6 "CONN HEADER LO-PRO 16POS AU SMD" H 5800 3100 60  0001 C CNN "Description"
-	1    5500 2350
-	1    0    0    -1
-$EndComp
 Wire Wire Line
 	3550 2300 3750 2300
@@
 Text Label 8800 3100 0    60   ~ 0
 RESET
+$Comp
+L HEADER_02X08_SMD P8
+U 1 1 56D96A90
+P 4550 1350
+F 0 "P8" H 4550 1800 50  0000 C CNN
+F 1 "HEADER_02X08_SMD" V 4550 1350 50  0000 C CNN
+F 2 "power_switch_controller:HEADER_02x08_SMD" H 4550 150 60  0001 C CNN
+F 3 "" H 4550 150 60  0000 C CNN
+F 4 "digikey" H 4650 1900 60  0001 C CNN "Vendor"
+F 5 "S9187-ND" H 4750 2000 60  0001 C CNN "PartNumber"
+F 6 "CONN HEADR 2.54MM 16POS GOLD SMD" H 4850 2100 60  0001 C CNN "Description"
+	1    4550 1350
+	1    0    0    -1
+$EndComp
+$Comp
+L HEADER_02X08_SMD P9
+U 1 1 56D96E95
+P 4550 2350
+F 0 "P9" H 4550 2800 50  0000 C CNN
+F 1 "HEADER_02X08_SMD" V 4550 2350 50  0000 C CNN
+F 2 "power_switch_controller:HEADER_02x08_SMD" H 4550 1150 60  0001 C CNN
+F 3 "" H 4550 1150 60  0000 C CNN
+F 4 "digikey" H 4650 2900 60  0001 C CNN "Vendor"
+F 5 "S9187-ND" H 4750 3000 60  0001 C CNN "PartNumber"
+F 6 "CONN HEADR 2.54MM 16POS GOLD SMD" H 4850 3100 60  0001 C CNN "Description"
+	1    4550 2350
+	1    0    0    -1
+$EndComp
+$Comp
+L HEADER_02X08_SMD P10
+U 1 1 56D970C5
+P 5500 1350
+F 0 "P10" H 5500 1800 50  0000 C CNN
+F 1 "HEADER_02X08_SMD" V 5500 1350 50  0000 C CNN
+F 2 "power_switch_controller:HEADER_02x08_SMD" H 5500 150 60  0001 C CNN
+F 3 "" H 5500 150 60  0000 C CNN
+F 4 "digikey" H 5600 1900 60  0001 C CNN "Vendor"
+F 5 "S9187-ND" H 5700 2000 60  0001 C CNN "PartNumber"
+F 6 "CONN HEADR 2.54MM 16POS GOLD SMD" H 5800 2100 60  0001 C CNN "Description"
+	1    5500 1350
+	1    0    0    -1
+$EndComp
+$Comp
+L HEADER_02X08_SMD P11
+U 1 1 56D971A8
+P 5500 2350
+F 0 "P11" H 5500 2800 50  0000 C CNN
+F 1 "HEADER_02X08_SMD" V 5500 2350 50  0000 C CNN
+F 2 "power_switch_controller:HEADER_02x08_SMD" H 5500 1150 60  0001 C CNN
+F 3 "" H 5500 1150 60  0000 C CNN
+F 4 "digikey" H 5600 2900 60  0001 C CNN "Vendor"
+F 5 "S9187-ND" H 5700 3000 60  0001 C CNN "PartNumber"
+F 6 "CONN HEADR 2.54MM 16POS GOLD SMD" H 5800 3100 60  0001 C CNN "Description"
+	1    5500 2350
+	1    0    0    -1
+$EndComp
 $EndSCHEMATC
