File: pcb/mega/power_switch_controller_mega.kicad_pcb (KiCad board)
At the start: 2 copper layers, 118.1 x 55.1 mm, 58 parts, among them P1 PWR_JACK_2.5x5.5, P10 HEADER_02X08_SMD, P11 HEADER_02X08_SMD, P2 HEADER_01X03_SMD_RA, P3 HEADER_01X03_SMD_RA, P4 HEADER_01X03_SMD_RA, P5 HEADER_01X03_SMD_RA, P6 HEADER_01X02_SMD_RA, P7 BNC_DOUBLE_RA, P8 HEADER_02X08_SMD, P9 HEADER_02X08_SMD, SW1 SPST_SLIDE_AS, U1 TLE7230R, U2 TLE7230R, U3 TLE7230R, U4 TLE7230R

Commit message: Create mega pcb.
Parts:
- ARDUINO1: footprint power_switch_controller:ARDUINO_MEGA_SHIELD -> power_switch_controller_mega:ARDUINO_MEGA_SHIELD
- C1, C2, C3, C4, C5, C6, C7: footprint power_switch_controller:SM1210 -> power_switch_controller_mega:SM1210
- D1, D10, D11, D12, D13, D14, D15, D16, D17, D18, D19, D2, D20, D21, D22, D23, D24, D25, D26, D27, D28, D29, D3, D30, D31, D32, D33, D4, D5, D6, D7, D8, D9: footprint power_switch_controller:LED_555-3XXX -> power_switch_controller_mega:LED_555-3XXX
- P1: footprint power_switch_controller:DCJACK_2PIN_HIGHCURRENT -> power_switch_controller_mega:DCJACK_2PIN_HIGHCURRENT
- P10, P11, P8, P9: footprint power_switch_controller:HEADER_02x08_SMD -> power_switch_controller_mega:HEADER_02x08_SMD
- P2, P3, P4, P5: footprint power_switch_controller:Header_3_Pin_SMD_RA -> power_switch_controller_mega:Header_3_Pin_SMD_RA
- P6: footprint power_switch_controller:Header_2_Pin_SMD_RA -> power_switch_controller_mega:Header_2_Pin_SMD_RA
- P7: footprint power_switch_controller:BNC_DOUBLE -> power_switch_controller_mega:BNC_DOUBLE
- REG1: footprint power_switch_controller:DC_DC_CONV_R78C -> power_switch_controller_mega:DC_DC_CONV_R78C
- SW1: footprint power_switch_controller:SPST_SLIDE_AS -> power_switch_controller_mega:SPST_SLIDE_AS
- U1, U2, U3, U4: footprint power_switch_controller:PG-DSO-36 -> power_switch_controller_mega:PG-DSO-36
Other:
- board text added: "Janelia Modular Device power_switch_controller_mega model_number: 1110 03/2016 ver 1.5"
- board text removed: "Janelia Modular Device power_switch_controller model_number: 1110 03/2016 ver 1.5"

Commit message: Progress towards mega pcb 1.6.
Parts:
- removed D10, D11, D12, D13, D14, D15, D16, D17, D18, D19, D2, D20, D21, D22, D23, D24, D25, D26, D27, D28, D29, D3, D30, D31, D32, D33, D4, D5, D6, D7, D8, D9: LED_24V, power_switch_controller_mega:LED_555-3XXX
- added L1: LED_24V, power_switch_controller_mega:LED_555-3XXX, F.Cu at (200.0, 109.2)
- added L10: LED_24V, power_switch_controller_mega:LED_555-3XXX, F.Cu at (135.9, 98.4)
- added L11: LED_24V, power_switch_controller_mega:LED_555-3XXX, F.Cu at (133.3, 98.4)
- added L12: LED_24V, power_switch_controller_mega:LED_555-3XXX, F.Cu at (130.8, 98.4)
- added L13: LED_24V, power_switch_controller_mega:LED_555-3XXX, F.Cu at (128.3, 98.4)
- added L14: LED_24V, power_switch_controller_mega:LED_555-3XXX, F.Cu at (125.7, 98.4)
- added L15: LED_24V, power_switch_controller_mega:LED_555-3XXX, F.Cu at (123.2, 98.4)
- added L16: LED_24V, power_switch_controller_mega:LED_555-3XXX, F.Cu at (120.7, 98.4)
- added L17: LED_24V, power_switch_controller_mega:LED_555-3XXX, F.Cu at (118.1, 98.4)
- added L18: LED_24V, power_switch_controller_mega:LED_555-3XXX, F.Cu at (171.4, 121.3)
- added L19: LED_24V, power_switch_controller_mega:LED_555-3XXX, F.Cu at (168.9, 121.3)
- added L2: LED_24V, power_switch_controller_mega:LED_555-3XXX, F.Cu at (171.4, 98.4)
- added L20: LED_24V, power_switch_controller_mega:LED_555-3XXX, F.Cu at (166.4, 121.3)
- added L21: LED_24V, power_switch_controller_mega:LED_555-3XXX, F.Cu at (163.8, 121.3)
- added L22: LED_24V, power_switch_controller_mega:LED_555-3XXX, F.Cu at (161.3, 121.3)
- added L23: LED_24V, power_switch_controller_mega:LED_555-3XXX, F.Cu at (158.8, 121.3)
- added L24: LED_24V, power_switch_controller_mega:LED_555-3XXX, F.Cu at (156.2, 121.3)
- added L25: LED_24V, power_switch_controller_mega:LED_555-3XXX, F.Cu at (153.7, 121.3)
- added L26: LED_24V, power_switch_controller_mega:LED_555-3XXX, F.Cu at (135.9, 121.3)
- added L27: LED_24V, power_switch_controller_mega:LED_555-3XXX, F.Cu at (133.3, 121.3)
- added L28: LED_24V, power_switch_controller_mega:LED_555-3XXX, F.Cu at (130.8, 121.3)
- added L29: LED_24V, power_switch_controller_mega:LED_555-3XXX, F.Cu at (128.3, 121.3)
- added L3: LED_24V, power_switch_controller_mega:LED_555-3XXX, F.Cu at (168.9, 98.4)
- added L30: LED_24V, power_switch_controller_mega:LED_555-3XXX, F.Cu at (125.7, 121.3)
- added L31: LED_24V, power_switch_controller_mega:LED_555-3XXX, F.Cu at (123.2, 121.3)
- added L32: LED_24V, power_switch_controller_mega:LED_555-3XXX, F.Cu at (120.7, 121.3)
- added L33: LED_24V, power_switch_controller_mega:LED_555-3XXX, F.Cu at (118.1, 121.3)
- added L4: LED_24V, power_switch_controller_mega:LED_555-3XXX, F.Cu at (166.4, 98.4)
- added L5: LED_24V, power_switch_controller_mega:LED_555-3XXX, F.Cu at (163.8, 98.4)
- added L6: LED_24V, power_switch_controller_mega:LED_555-3XXX, F.Cu at (161.3, 98.4)
- added L7: LED_24V, power_switch_controller_mega:LED_555-3XXX, F.Cu at (158.8, 98.4)
- added L8: LED_24V, power_switch_controller_mega:LED_555-3XXX, F.Cu at (156.2, 98.4)
- added L9: LED_24V, power_switch_controller_mega:LED_555-3XXX, F.Cu at (153.7, 98.4)
- D1: value LED_24V -> diode_schottky_45V_10A; footprint power_switch_controller_mega:LED_555-3XXX -> power_switch_controller_mega:CFP15
- REG1: value CONV_DC_DC_12V_1A -> CONV_DC_DC_9V_1A
- moved D1 19.7 mm to (201.9, 113.7), turned to 90 degrees
- moved SW1 18.5 mm to (201.3, 94.0), turned to 270 degrees
- moved C1 10.2 mm to (201.3, 98.4)
Connections:
- ARDUINO1 pad 45: (no net) -> /IN
- D1 pad 1: /LED_PWR -> VCC
- D1 pad 2: GND -> VAA
- P6 pad 2: VAA -> VCC
- U1 pad 12: GND -> +5V
- U1 pad 13: GND -> /IN
- U1 pad 6: GND -> +5V
- U1 pad 7: GND -> +5V
- U2 pad 12: GND -> +5V
- U2 pad 13: GND -> /IN
- U2 pad 6: GND -> +5V
- U2 pad 7: GND -> +5V
- U3 pad 12: GND -> +5V
- U3 pad 13: GND -> /IN
- U3 pad 6: GND -> +5V
- U3 pad 7: GND -> +5V
- U4 pad 12: GND -> +5V
- U4 pad 13: GND -> /IN
- U4 pad 6: GND -> +5V
- U4 pad 7: GND -> +5V
Routing:
- net /IN: track 0.00 -> 112.8 mm, vias 0 -> 4
- net GND: track 558.3 -> 478.2 mm
- net /BNC_A: track 91.3 -> 118.6 mm, vias 0 -> 1
- net /CS: track 96.8 -> 114.8 mm
- net /OUT26: track 28.1 -> 44.2 mm
- net /RESET: track 97.9 -> 111.8 mm, vias 1 -> 3
- net VAA: track 217.8 -> 229.1 mm, vias 1 -> 0
- net /SO2: track 61.2 -> 52.4 mm, vias 0 -> 2
- net VCC: track 0.00 -> 7.40 mm
- net /MISO: track 62.2 -> 68.6 mm
- net /MOSI: track 39.8 -> 45.7 mm
- net /LED_PWR: track 207.8 -> 202.0 mm
- net /SO1: track 41.1 -> 36.1 mm, vias 0 -> 2
- net /SCK: track 112.7 -> 116.0 mm, vias 5 -> 4
- net +5V: track 216.2 -> 214.3 mm, vias 4 -> 3
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- removed copper zone on B.Cu, net GND
- removed copper zone on F.Cu, net VAA
Other:
- board text added: "+12-42VDC"
- board text added: "9V"
- board text added: "Janelia Modular Device power_switch_controller model_number: 1110 06/2016 ver 1.6 mega"
- board text removed: "+24VDC"
- board text removed: "12V"
- board text removed: "Janelia Modular Device power_switch_controller_mega model_number: 1110 03/2016 ver 1.5"

Commit message: Finished pcb 1.6.
Parts:
- turned SW1 to 90 degrees
Routing:
- net +5V: track 214.3 -> 257.5 mm, vias 3 -> 2
- net GND: track 478.2 -> 519.6 mm, vias 1 -> 2
- net /SO1: track 36.1 -> 71.1 mm, vias 2 -> 0
- net /SCK: track 116.0 -> 148.2 mm, vias 4 -> 2
- net /BNC_A: track 118.6 -> 91.3 mm, vias 1 -> 0
- net VAA: track 229.1 -> 253.8 mm, vias 0 -> 1
- net /OUT8: track 22.3 -> 41.1 mm, vias 1 -> 0
- net /OUT26: track 44.2 -> 27.9 mm, vias 0 -> 1
- net /OUT15: track 28.2 -> 44.3 mm
- net /RX3: track 66.1 -> 81.9 mm, vias 0 -> 1
- net /OUT27: track 30.6 -> 45.2 mm, vias 1 -> 0
- net /CS: track 114.8 -> 104.4 mm, vias 2 -> 3
- net /IN: track 112.8 -> 121.3 mm, vias 4 -> 2
- net /OUT9: track 26.1 -> 34.6 mm, vias 1 -> 0
- net /OUT13: track 20.8 -> 28.4 mm
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- added copper zone on B.Cu, net GND
- added copper zone on F.Cu, net VAA

Commit message: Progess towards mega pcb1.7.
Routing:
- net GND: track 519.6 -> 0.00 mm, vias 2 -> 0
- net +5V: track 257.5 -> 0.00 mm, vias 2 -> 0
- net VAA: track 253.8 -> 0.00 mm, vias 1 -> 0
- net /LED_PWR: track 205.2 -> 0.00 mm
- net /SCK: track 148.2 -> 0.00 mm, vias 2 -> 0
- net /IN: track 121.3 -> 0.00 mm, vias 2 -> 0
- net /CS: track 104.4 -> 0.00 mm, vias 3 -> 0
- net /RESET: track 104.2 -> 0.00 mm, vias 2 -> 0
- net /BNC_A: track 91.3 -> 0.00 mm
- net /TX3: track 85.0 -> 0.00 mm
- net /RX3: track 81.9 -> 0.00 mm, vias 1 -> 0
- net /SO1: track 71.1 -> 0.00 mm
- net /RX0: track 70.0 -> 0.00 mm
- net /MISO: track 62.1 -> 0.00 mm, vias 1 -> 0
- net /TX0: track 58.4 -> 0.00 mm
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- removed copper zone on B.Cu, net GND
- removed copper zone on F.Cu, net VAA
Other:
- board text added: "Janelia Modular Device power_switch_controller model_number: 1110 07/2016 ver 1.7 mega"
- board text removed: "Janelia Modular Device power_switch_controller model_number: 1110 06/2016 ver 1.6 mega"
