File: pcb/teensy/power_switch_controller_teensy.sch (KiCad schematic (older format))
At the start: 20 parts, among them P1 PWR_JACK_2.5x5.5_SMD_RA, P2 HEADER_01X03_SMD_RA, P3 HEADER_01X03_SMD_RA, P4 HEADER_01X03_SMD_RA, P5 BNC_DOUBLE_RA, P6 HEADER_01X02_SMD_RA, P7 HEADER_01X02_SMD_RA, SW1 KT_SWITCH

Commit message: Progress towards teensy v1.0.
Parts:
- removed C1, C2, C3, C4, C5: 10uF, power_switch_controller_teensy:SM1210, symbol 10uF
- removed D1, D2: diode_schottky_15V_1A, power_switch_controller_teensy:DO-214BA, symbol diode_schottky_15V_1A
- removed D3, D4: diode_schottky_45V_10A, power_switch_controller_teensy:CFP15, symbol diode_schottky_45V_10A
- removed P1: PWR_JACK_2.5x5.5_SMD_RA, power_switch_controller_teensy:DCJACK_2PIN_HIGHCURRENT_SMD_RA, symbol PWR_JACK_2.5x5.5_SMD_RA
- removed P2, P3, P4: HEADER_01X03_SMD_RA, power_switch_controller_teensy:Header_3_Pin_SMD_RA, symbol HEADER_01X03_SMD_RA
- removed P5: BNC_DOUBLE_RA, power_switch_controller_teensy:BNC_DOUBLE, symbol BNC_DOUBLE_RA
- removed P6, P7: HEADER_01X02_SMD_RA, power_switch_controller_teensy:Header_2_Pin_SMD_RA, symbol HEADER_01X02_SMD_RA
- removed REG1: CONV_DC_DC_5V_1A, power_switch_controller_teensy:DC_DC_CONV_R78C, symbol CONV_DC_DC_5V_1A
- removed SW1: KT_SWITCH, power_switch_controller_teensy:KT_SWITCH, symbol KT_SWITCH
- removed TEENSY1: TEENSY_3_2, power_switch_controller_teensy:TEENSY_3, symbol TEENSY_3_2
- added C?: 0.1uF, power_switch_controller_teensy:SM1210, symbol 0.1uF
- added L1, L? (x8): LED_24V, power_switch_controller_teensy:LED_555-3XXX, symbol LED_24V
- added P?: HEADER_02X08_SMD, power_switch_controller_teensy:HEADER_02x08_SMD, symbol HEADER_02X08_SMD
- added SW1: SPST_SLIDE_AS, power_switch_controller_teensy:SPST_SLIDE_AS, symbol SPST_SLIDE_AS
- added U?: TLE7230R, power_switch_controller_teensy:PG-DSO-36, symbol TLE7230R
Connections:
- net GND: now also C?.2, L1.2 (K), U?.1 (GND), U?.18 (GND), U?.19 (GND), U?.36 (GND)
- net VDD: now also P?.1 (P1), P?.11 (P11), P?.13 (P13), P?.15 (P15), P?.3 (P3), P?.5 (P5), P?.7 (P7), P?.9 (P9), SW1.1
- net VEE: now also C?.1, U?.12 (IN3), U?.25 (VDO), U?.6 (IN1), U?.7 (IN2), U?.8 (VS)
- net 3V3: no longer names the net of MDT1.3V3 (3.3v_(250_mA_max))
- net AGND: no longer names the net of MDT1.AGND
- net AREF: no longer names the net of MDT1.AREF
- net D10 renamed CS
- net CS: now also U?.10 (CS)
- net D11 renamed MOSI
- net MOSI: now also U?.29 (SI)
- net D12 renamed MISO
- net MISO: now also U?.27 (SO)
- net D13 renamed SCK
- net SCK: now also U?.28 (SCLK)
- net D14: no longer names the net of MDT1.14 (D14/A0/SCKB)
- net D15: no longer names the net of MDT1.15 (D15/A1/TOUCH/CSB)
- net D16: no longer names the net of MDT1.16 (D16/A2/TOUCH)
- net D17: no longer names the net of MDT1.17 (D17/A3/TOUCH)
- net D18: no longer names the net of MDT1.18 (D18/A4/SDA0/TOUCH)
- net D19: no longer names the net of MDT1.19 (D19/A5/SCL0/TOUCH)
- net D2 renamed RESET
- net RESET: now also U?.9 (RST)
- net D20: no longer names the net of MDT1.20 (D20/A6/PWM/CSB)
- net D21: no longer names the net of MDT1.21 (D21/A7/PWM/RX1B/CSB)
- net D22: no longer names the net of MDT1.22 (D22/A8/TOUCH/PWM/ICP/I2STX)
- net D23: no longer names the net of MDT1.23 (D23/A9/TOUCH/PWM/ICP/I2SLRCLK)
- net D24: no longer names the net of MDT1.24 (D24/ICP/I2SBCLKB)
- net D25: no longer names the net of MDT1.25 (D25/PWM/TOUCH/I2SLRCLK2)
- net D28: no longer names the net of MDT1.28 (D28/A17/I2SMCLKB)
- net D29: no longer names the net of MDT1.29 (D29/A18/SCL1)
- net D3 renamed PWM
- net PWM: now also U?.13 (IN4)
- net D30: no longer names the net of MDT1.30 (D30/A19/SDA1)
- net D4: no longer names the net of MDT1.4 (D4/PWM/CANRX)
- net D5: no longer names the net of MDT1.5 (D5/PWM/TX1B)
- net D6: no longer names the net of MDT1.6 (D6/PWM)
- net D9: no longer names the net of MDT1.9 (D9/RX2/PWM/ICP/CSB/I2SBCLK)
- net DAC: no longer names the net of MDT1.DAC (A14/DAC)
- new net LED_PWR: L1.1 (A), SW1.3
- new net OUT0: P?.2 (P2), U?.4 (OUT1)
- new net OUT1: P?.4 (P4), U?.5 (OUT2)
- new net OUT2: P?.6 (P6), U?.14 (OUT3)
- new net OUT3: P?.8 (P8), U?.15 (OUT4)
- new net OUT4: P?.10 (P10), U?.22 (OUT5)
- new net OUT5: P?.12 (P12), U?.23 (OUT6)
- new net OUT6: P?.14 (P14), U?.32 (OUT7)
- new net OUT7: P?.16 (P16), U?.33 (OUT8)
- no-connect marks 5 -> 25
Other:
- moved on the sheet: MDT1

Commit message: More progress towards v1.0.
Parts:
- removed MDT1: MODULAR_DEVICE_TEENSY, power_switch_controller_teensy:MODULAR_DEVICE_TEENSY, symbol MODULAR_DEVICE_TEENSY
- added C1: 10uF, power_switch_controller_teensy:SM1210, symbol 10uF
- added MDT1: MODULAR_DEVICE_TEENSY_MALE, power_switch_controller_teensy:MODULAR_DEVICE_TEENSY, symbol MODULAR_DEVICE_TEENSY_MALE
- gave numbers to parts that had none: 11
Connections:
- net CS: now also MDT1.10 (D10/TX2/CS/PWM/ICP)
- net GND: now also C1.2, MDT1.GND
- net LED_PWR: now also L2.1 (A), L3.1 (A), L4.1 (A), L5.1 (A), L6.1 (A), L7.1 (A), L8.1 (A), L9.1 (A)
- net MISO: now also MDT1.12 (D12/DIN)
- net MOSI: now also MDT1.11 (D11/DOUT/I2SMCLK)
- net OUT0: now also L2.2 (K)
- net OUT1: now also L3.2 (K)
- net OUT2: now also L4.2 (K)
- net OUT3: now also L5.2 (K)
- net OUT4: now also L6.2 (K)
- net OUT5: now also L7.2 (K)
- net OUT6: now also L8.2 (K)
- net OUT7: now also L9.2 (K)
- net PWM: now also MDT1.3 (D3/PWM/CANTX)
- net RESET: now also MDT1.2 (D2)
- net SCK: now also MDT1.13 (D13/LED/SCK/I2SRX)
- net VDD: now also C1.1, MDT1.VDD (VDD_(+9-42VDC))
- net VEE: now also MDT1.VEE (VEE_(+4-5VDC))

Commit message: Finished pcb v1.1.
Parts:
- MDT1: footprint power_switch_controller_teensy:MODULAR_DEVICE_TEENSY -> power_switch_controller_teensy:MODULAR_DEVICE_TEENSY_MALE
Changed lines of the file:
@@
 LIBS:components
 LIBS:power_switch_controller_teensy
-LIBS:power_switch_controller_teensy-cache
 EELAYER 25 0
 EELAYER END
@@
 Title "power_switch_controller_teensy"
 Date ""
-Rev "1.0"
+Rev "1.1"
 Comp "Janelia"
 Comment1 ""
@@
 $Comp
 L MODULAR_DEVICE_TEENSY_MALE MDT1
-U 1 1 578F97F5
+U 1 1 57A8C92C
 P 2600 1600
 F 0 "MDT1" H 2600 2597 60  0000 C CNN
 F 1 "MODULAR_DEVICE_TEENSY_MALE" H 2600 2491 60  0000 C CNN
-F 2 "power_switch_controller_teensy:MODULAR_DEVICE_TEENSY" H 2600 2650 60  0001 C CNN
+F 2 "power_switch_controller_teensy:MODULAR_DEVICE_TEENSY_MALE" H 2600 2650 60  0001 C CNN
 F 3 "" H 2650 4350 60  0000 C CNN
 F 4 "digikey" H 2600 2750 60  0001 C CNN "Vendor"
